File: matrix_main_board.sch (EAGLE design)
At the start: 148 parts, among them IC1 MKE02_44PIN, IC2 24AA01SM, IC3 74HC595D, IC4 74HC595D, IC5 74HC595D, IC6 74HC595D, IC7 NPIC6C596, IC8 NPIC6C596, IC9 W25Q128

Commit message: 3v3/rp2010
Parts:
- removed C1, C19, C21, C4: (no value), rcl:C-EUC0805
- removed C11, C2: 18p, rcl:C-EUC0805
- removed GD3, GD5: (no value), pinhead:PINHD-1X1
- removed IC1: MKE02_44PIN, jason_eagle6:MKE02_44PIN
- removed PD6, PD7, PH2: TPTP17R, testpad:TPTP17R
- removed R5, R6: (no value), rcl:R-EU_R0805
- removed XTL1: 20m, crystal:CRYSTALHC49S
- added D+, D-: (no value), pinhead:PINHD-1X1
- added TP1, TP2: TPTP07SQ, testpad:TPTP07SQ
- C14, C15, C17, C18, C20, C22, C23, C24, C25, C26, C27: device rcl:C-EUC0805 -> rcl:C-EUC0603K
- C16: value 18p -> 100n; device rcl:C-EUC0805 -> resistor:C-EUC0603
- R45: device rcl:R-EU_R0805 -> rcl:R-EU_R0603
Connections:
- removed net +5V: C1.2, C10.2, C12.+, C13.+, C3.2, C4.2, C5.2, C6.2, C7.2, C8.2, C9.2, IC1.VDD, IC1.VDD1, IC1.VDDA/REFH, IC2.VCC, IC3A.SCL, IC3P.VCC, IC4A.SCL, IC4P.VCC, IC5A.SCL, IC5P.VCC, IC6A.SCL, IC6P.VCC, IC7.MR#, IC7.VCC, IC8.MR#, IC8.VCC, R1.2, R2.2, R3.2, R4.2, R42.2, R43.2, R44.2, R5.2, VCC.1, VCC1.1, VCC2.1
- removed net N$44: U$1.TESTEN
- removed net N$45: U$1.SWCLK
- removed net N$46: U$1.SWDIO
- removed net N$47: U$1.RUN
- removed net NRESET: IC1.PTA5, R3.1, RESET.1
- removed net PTD6: IC1.PTD6, PD6.TP
- removed net PTD7: IC1.PTD7, PD7.TP
- removed net PTH2: IC1.PTH2, PH2.TP
- removed net SWDCLK: IC1.PTC4, R5.1, SWD_CLK.1
- removed net SWDIO: IC1.PTA4, R4.1, SWD_DAT.1
- removed net VCC: C16.2, IC9.VCC, R46.1
- new net N$25: D-.1, R4.2
- new net N$26: TP2.TP, U$1.TESTEN
- new net SWD_CLK: SWD_CLK.1, U$1.SWCLK
- new net SWD_DAT: SWD_DAT.1, U$1.SWDIO
- new net SWD_RESET: RESET.1, U$1.RUN
- net +3V3: now also C10.2, C12.+, C13.+, C16.2, C3.2, C5.2, C6.2, C7.2, C8.2, C9.2, IC2.VCC, IC3A.SCL, IC3P.VCC, IC4A.SCL, IC4P.VCC, IC5A.SCL, IC5P.VCC, IC6A.SCL, IC6P.VCC, IC7.MR#, IC7.VCC, IC8.MR#, IC8.VCC, IC9.VCC, R1.2, R2.2, R42.2, R43.2, R44.2, R46.1, VCC.1, VCC1.1; no longer C19.2, C21.2
- net AUXIN: now also U$1.GPIO29/ADC3; no longer IC1.PTC7, U$1.GPIO19
- net AUXOUT: now also U$1.GPIO1; no longer IC1.PTA7, U$1.GPIO18
- net D_ACK: now also U$1.GPIO2; no longer IC1.PTB2
- net D_ADT: now also U$1.GPIO5; no longer IC1.PTB3, U$1.GPIO15
- net D_ARK: now also U$1.GPIO3; no longer IC1.PTC0, U$1.GPIO13
- net D_ENA: now also U$1.GPIO4; no longer IC1.PTA1, U$1.GPIO22
- net D_KCK: now also U$1.GPIO24; no longer IC1.PTC1, U$1.GPIO12, U$1.GPIO14
- net D_KDT: now also U$1.GPIO23; no longer IC1.PTD5, U$1.GPIO11
- net ENC1: now also U$1.GPIO20; no longer IC1.PTD1, U$1.GPIO0
- net ENC2: now also U$1.GPIO19; no longer IC1.PTD0, U$1.GPIO1
- net GATE1: now also U$1.GPIO11; no longer IC1.PTD2, U$1.GPIO7
- net GATE2: now also U$1.GPIO10; no longer IC1.PTD3, U$1.GPIO8
- net GATE3: no longer IC1.PTD4
- net GATE4: now also U$1.GPIO8; no longer IC1.PTA6, U$1.GPIO10
- net GND: no longer C1.1, C11.1, C19.1, C2.1, C21.1, C4.1, GD3.1, GD5.1, IC1.VSS, IC1.VSS1, IC1.VSSA/VSS
- net I2C0SCL: now also U$1.GPIO13; no longer IC1.PTA3, U$1.GPIO21
- net I2C0SDA: now also U$1.GPIO12; no longer IC1.PTA2, U$1.GPIO20
- net I2C1SCL: no longer IC1.PTE1
- net I2C1SDA: no longer IC1.PTE0
- net KEY_READ1: now also U$1.GPIO22; no longer IC1.PTC6, U$1.GPIO28/ADC2
- net KEY_READ2: now also U$1.GPIO21; no longer IC1.PTB4, U$1.GPIO29/ADC3
- net LED1: now also U$1.GPIO16; no longer IC1.PTB5, U$1.GPIO4
- net LED2: now also U$1.GPIO17; no longer IC1.PTC3, U$1.GPIO5
- net LED3: now also U$1.GPIO18; no longer IC1.PTC2, U$1.GPIO6
- net MIDIRX: now also U$1.GPIO7; no longer IC1.PTB0, U$1.GPIO17
- net MIDITX: now also U$1.GPIO6; no longer IC1.PTB1, U$1.GPIO16
- net N$4: now also VCC2.1; no longer C2.2, IC1.PTB7, R6.2, XTL1.2
- net N$5: now also D+.1, R3.2; no longer C11.2, IC1.PTB6, R6.1, XTL1.1
- net N$65: now also TP1.TP
- net OFF_SW: now also U$1.GPIO14; no longer IC1.PTE7, U$1.GPIO2
- net PWR_CTRL: now also U$1.GPIO28/ADC2; no longer IC1.PTE2, U$1.GPIO3
- net SYNCIN: now also U$1.GPIO0; no longer IC1.PTA0, U$1.GPIO23
- net SYNCOUT: now also U$1.GPIO15; no longer IC1.PTC5, U$1.GPIO24
- net USB_DM: now also R4.1
- net USB_DP: now also R3.1
Other:
- moved on the sheet: C14, C15, C17, C18, C20, C22, C23, C24, C25, C26, C27, Q1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

Commit message: Rolling back RP2040 changes
Parts:
- removed C14, C15: 18p, rcl:C-EUC0603K
- removed C16: 100n, resistor:C-EUC0603
- removed C17, C18, C20, C22, C23, C26, C27: (no value), rcl:C-EUC0603K
- removed C24, C25: 1u, rcl:C-EUC0603K
- removed D+, D-: (no value), pinhead:PINHD-1X1
- removed IC9: W25Q128, jason_eagle6:W25Q128
- removed Q1: (no value), adafruit:CRYSTALCTS406
- removed R45: (no value), rcl:R-EU_R0603
- removed R46, R47: (no value), rcl:R-EU_R0805
- removed TP1, TP2: TPTP07SQ, testpad:TPTP07SQ
- removed U$1: RP2040, jason_eagle6:RP2040
- added C1, C4: (no value), rcl:C-EUC0805
- added C11, C2: 18p, rcl:C-EUC0805
- added GD3, GD5: (no value), pinhead:PINHD-1X1
- added IC1: MKE02_44PIN, jason_eagle6:MKE02_44PIN
- added PD6, PD7, PH2: TPTP17R, testpad:TPTP17R
- added R5, R6: (no value), rcl:R-EU_R0805
- added XTL1: 20m, crystal:CRYSTALHC49S
Connections:
- removed net +1V1: C25.2, C26.2, C27.2, U$1.DVDD1, U$1.DVDD2, U$1.VREG_VOUT
- removed net +3V3: C10.2, C12.+, C13.+, C16.2, C17.2, C18.2, C20.2, C22.2, C23.2, C24.2, C3.2, C5.2, C6.2, C7.2, C8.2, C9.2, IC2.VCC, IC3A.SCL, IC3P.VCC, IC4A.SCL, IC4P.VCC, IC5A.SCL, IC5P.VCC, IC6A.SCL, IC6P.VCC, IC7.MR#, IC7.VCC, IC8.MR#, IC8.VCC, IC9.VCC, R1.2, R2.2, R42.2, R43.2, R44.2, R46.1, U$1.ADC_AVDD, U$1.IOVDD1, U$1.IOVDD2, U$1.IOVDD3, U$1.IOVDD4, U$1.IOVDD5, U$1.IOVDD6, U$1.USB_VDD, U$1.VREG_VIN, VCC.1, VCC1.1
- removed net N$10: C14.2, Q1.2, U$1.XIN
- removed net N$12: C15.2, Q1.1, R45.2
- removed net N$15: R45.1, U$1.XOUT
- removed net N$25: D-.1, R4.2
- removed net N$26: TP2.TP, U$1.TESTEN
- removed net N$65: TP1.TP, U$1.GPIO25
- removed net QSPI_CSN: IC9.CS#, R46.2, R47.2, U$1.QSPI_SS#
- removed net QSPI_SCLK: IC9.CLK, U$1.QSPI_SCLK
- removed net QSPI_SD0: IC9.DIO/IO0, U$1.QSPI_SD0
- removed net QSPI_SD1: IC9.DO/IO1, U$1.QSPI_SD1
- removed net QSPI_SD2: IC9.WP#/IO2, U$1.QSPI_SD2
- removed net QSPI_SD3: IC9.RES#/IO3, U$1.QSPI_SD3
- removed net SWD_CLK: SWD_CLK.1, U$1.SWCLK
- removed net SWD_DAT: SWD_DAT.1, U$1.SWDIO
- removed net SWD_RESET: RESET.1, U$1.RUN
- removed net USB_DM: R4.1, U$1.USB_DM
- removed net USB_DP: R3.1, U$1.USB_DP
- new net +5V: C1.2, C10.2, C12.+, C13.+, C3.2, C4.2, C5.2, C6.2, C7.2, C8.2, C9.2, IC1.VDD, IC1.VDD1, IC1.VDDA/REFH, IC2.VCC, IC3A.SCL, IC3P.VCC, IC4A.SCL, IC4P.VCC, IC5A.SCL, IC5P.VCC, IC6A.SCL, IC6P.VCC, IC7.MR#, IC7.VCC, IC8.MR#, IC8.VCC, R1.2, R2.2, R3.2, R4.2, R42.2, R43.2, R44.2, R5.2, VCC.1, VCC1.1, VCC2.1
- new net NRESET: IC1.PTA5, R3.1, RESET.1
- new net PTD6: IC1.PTD6, PD6.TP
- new net PTD7: IC1.PTD7, PD7.TP
- new net PTH2: IC1.PTH2, PH2.TP
- new net SWDCLK: IC1.PTC4, R5.1, SWD_CLK.1
- new net SWDIO: IC1.PTA4, R4.1, SWD_DAT.1
- net AUXIN: now also IC1.PTC7; no longer U$1.GPIO29/ADC3
- net AUXOUT: now also IC1.PTA7; no longer U$1.GPIO1
- net D_ACK: now also IC1.PTB2; no longer U$1.GPIO2
- net D_ADT: now also IC1.PTB3; no longer U$1.GPIO5
- net D_ARK: now also IC1.PTC0; no longer U$1.GPIO3
- net D_ENA: now also IC1.PTA1; no longer U$1.GPIO4
- net D_KCK: now also IC1.PTC1; no longer U$1.GPIO24
- net D_KDT: now also IC1.PTD5; no longer U$1.GPIO23
- net ENC1: now also IC1.PTD1; no longer U$1.GPIO20
- net ENC2: now also IC1.PTD0; no longer U$1.GPIO19
- net GATE1: now also IC1.PTD2; no longer U$1.GPIO11
- net GATE2: now also IC1.PTD3; no longer U$1.GPIO10
- net GATE3: now also IC1.PTD4; no longer U$1.GPIO9
- net GATE4: now also IC1.PTA6; no longer U$1.GPIO8
- net GND: now also C1.1, C11.1, C2.1, C4.1, GD3.1, GD5.1, IC1.VSS, IC1.VSS1, IC1.VSSA/VSS; no longer C14.1, C15.1, C16.1, C17.1, C18.1, C20.1, C22.1, C23.1, C24.1, C25.1, C26.1, C27.1, IC9.GND, U$1.GND
- net I2C0SCL: now also IC1.PTA3; no longer U$1.GPIO13
- net I2C0SDA: now also IC1.PTA2; no longer U$1.GPIO12
- net I2C1SCL: now also IC1.PTE1; no longer U$1.GPIO27/ADC1
- net I2C1SDA: now also IC1.PTE0; no longer U$1.GPIO26/ADC0
- net KEY_READ1: now also IC1.PTC6; no longer U$1.GPIO22
- net KEY_READ2: now also IC1.PTB4; no longer U$1.GPIO21
- net LED1: now also IC1.PTB5; no longer U$1.GPIO16
- net LED2: now also IC1.PTC3; no longer U$1.GPIO17
- net LED3: now also IC1.PTC2; no longer U$1.GPIO18
- net MIDIRX: now also IC1.PTB0; no longer U$1.GPIO7
- net MIDITX: now also IC1.PTB1; no longer U$1.GPIO6
- net N$4: now also C2.2, IC1.PTB7, R6.2, XTL1.2; no longer VCC2.1
- net N$5: now also C11.2, IC1.PTB6, R6.1, XTL1.1; no longer D+.1, R3.2
- net OFF_SW: now also IC1.PTE7; no longer R47.1, U$1.GPIO14
- net PWR_CTRL: now also IC1.PTE2; no longer U$1.GPIO28/ADC2
- net SYNCIN: now also IC1.PTA0; no longer U$1.GPIO0
- net SYNCOUT: now also IC1.PTC5; no longer U$1.GPIO15
Other:
- moved on the sheet: R3, R4

Commit message: dsfdfs
Parts:
- added C14, C15, C16: 18p, rcl:C-EUC0805
- added IC9: W25Q128, jason_eagle6:W25Q128
- added Q1: (no value), adafruit:CRYSTALCTS406
- added R45, R46, R47: (no value), rcl:R-EU_R0805
- added U1: RP2040, RP2040:RP2040
Connections:
- new net N$10: C14.2, Q1.2, U1.XIN
- new net N$12: C15.2, Q1.1, R45.2
- new net N$15: R45.1, U1.XOUT
- new net QSPI_CSN: IC9.CS#, R46.2, R47.2, U1.QSPI_CSN
- new net QSPI_SCLK: IC9.CLK, U1.QSPI_SCLK
- new net QSPI_SD0: IC9.DIO/IO0, U1.QSPI_SD0
- new net QSPI_SD1: IC9.DO/IO1, U1.QSPI_SD1
- new net QSPI_SD2: IC9.WP#/IO2, U1.QSPI_SD2
- new net QSPI_SD3: IC9.RES#/IO3, U1.QSPI_SD3
- new net VCC: C16.2, IC9.VCC, R46.1
- net GND: now also C14.1, C15.1, C16.1, IC9.GND, U1.GND
- net OFF_SW: now also R47.1
Changed lines of the file:
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@@
 <part name="R44" library="rcl" deviceset="R-EU_" device="R0805" value="4k7"/>
 <part name="P+14" library="supply1" deviceset="+5V" device=""/>
+<part name="U1" library="RP2040" deviceset="RP2040" device=""/>
+<part name="Q1" library="adafruit" deviceset="CRYSTAL" device="CTS406"/>
+<part name="R45" library="rcl" deviceset="R-EU_" device="R0805"/>
+<part name="C14" library="rcl" deviceset="C-EU" device="C0805" value="18p"/>
+<part name="C15" library="rcl" deviceset="C-EU" device="C0805" value="18p"/>
+<part name="GND14" library="supply1" deviceset="GND" device=""/>
+<part name="IC9" library="jason_eagle6" deviceset="W25Q128" device=""/>
+<part name="C16" library="rcl" deviceset="C-EU" device="C0805" value="18p"/>
+<part name="GND15" library="supply1" deviceset="GND" device=""/>
+<part name="P+12" library="supply1" deviceset="VCC" device=""/>
+<part name="R46" library="rcl" deviceset="R-EU_" device="R0805"/>
+<part name="P+15" library="supply1" deviceset="VCC" device=""/>
+<part name="R47" library="rcl" deviceset="R-EU_" device="R0805"/>
+<part name="GND16" library="supply1" deviceset="GND" device=""/>
 </parts>
 <sheets>
@@
 <instance part="R44" gate="G$1" x="134.62" y="154.94" rot="R90"/>
 <instance part="P+14" gate="1" x="129.54" y="175.26"/>
+<instance part="U1" gate="G$1" x="-2.54" y="-50.8"/>
+<instance part="Q1" gate="G$1" x="-45.72" y="-38.1" rot="R90"/>
+<instance part="R45" gate="G$1" x="-33.02" y="-40.64" rot="R180"/>
+<instance part="C14" gate="G$1" x="-53.34" y="-33.02" rot="R90"/>
+<instance part="C15" gate="G$1" x="-53.34" y="-43.18" rot="R90"/>
+<instance part="GND14" gate="1" x="-63.5" y="-43.18"/>
+<instance part="IC9" gate="G$1" x="147.32" y="-22.86"/>
+<instance part="C16" gate="G$1" x="147.32" y="-33.02" rot="R90"/>
+<instance part="GND15" gate="1" x="129.54" y="-38.1"/>
+<instance part="P+12" gate="VCC" x="170.18" y="0"/>
+<instance part="R46" gate="G$1" x="129.54" y="-5.08" rot="R270"/>
+<instance part="P+15" gate="VCC" x="129.54" y="5.08"/>
+<instance part="R47" gate="G$1" x="119.38" y="-12.7"/>
+<instance part="GND16" gate="1" x="25.4" y="-99.06"/>
 </instances>
 <busses>
@@
 <wire x1="-33.02" y1="162.56" x2="-33.02" y2="160.02" width="0.1524" layer="91"/>
 </segment>
+<segment>
+<pinref part="C14" gate="G$1" pin="1"/>
+<wire x1="-55.88" y1="-33.02" x2="-58.42" y2="-33.02" width="0.1524" layer="91"/>
+<wire x1="-58.42" y1="-33.02" x2="-58.42" y2="-38.1" width="0.1524" layer="91"/>
+<pinref part="C15" gate="G$1" pin="1"/>
+<wire x1="-58.42" y1="-38.1" x2="-58.42" y2="-43.18" width="0.1524" layer="91"/>
+<wire x1="-58.42" y1="-43.18" x2="-55.88" y2="-43.18" width="0.1524" layer="91"/>
+<pinref part="GND14" gate="1" pin="GND"/>
+<wire x1="-58.42" y1="-38.1" x2="-63.5" y2="-38.1" width="0.1524" layer="91"/>
+<wire x1="-63.5" y1="-38.1" x2="-63.5" y2="-40.64" width="0.1524" layer="91"/>
+<junction x="-58.42" y="-38.1"/>
+</segment>
+<segment>
+<pinref part="IC9" gate="G$1" pin="GND"/>
+<wire x1="132.08" y1="-25.4" x2="129.54" y2="-25.4" width="0.1524" layer="91"/>
+<wire x1="129.54" y1="-25.4" x2="129.54" y2="-33.02" width="0.1524" layer="91"/>
+<pinref part="C16" gate="G$1" pin="1"/>
+<wire x1="129.54" y1="-33.02" x2="144.78" y2="-33.02" width="0.1524" layer="91"/>
+<pinref part="GND15" gate="1" pin="GND"/>
+<wire x1="129.54" y1="-35.56" x2="129.54" y2="-33.02" width="0.1524" layer="91"/>
+<junction x="129.54" y="-33.02"/>
+</segment>
+<segment>
+<pinref part="U1" gate="G$1" pin="GND"/>
+<pinref part="GND16" gate="1" pin="GND"/>
+<wire x1="20.32" y1="-93.98" x2="25.4" y2="-93.98" width="0.1524" layer="91"/>
+<wire x1="25.4" y1="-93.98" x2="25.4" y2="-96.52" width="0.1524" layer="91"/>
+</segment>
 </net>
 <net name="N$122" class="0">
@@
 <wire x1="-40.64" y1="99.06" x2="-53.34" y2="99.06" width="0.1524" layer="91"/>
 <label x="-53.34" y="99.06" size="1.778" layer="95"/>
+</segment>
+<segment>
+<pinref part="R47" gate="G$1" pin="1"/>
+<wire x1="114.3" y1="-12.7" x2="106.68" y2="-12.7" width="0.1524" layer="91"/>
+<label x="99.06" y="-12.7" size="1.778" layer="95"/>
 </segment>
 </net>
@@
 </segment>
 </net>
+<net name="N$10" class="0">
+<segment>
+<pinref part="C14" gate="G$1" pin="2"/>
+<pinref part="Q1" gate="G$1" pin="2"/>
+<wire x1="-48.26" y1="-33.02" x2="-45.72" y2="-33.02" width="0.1524" layer="91"/>
+<wire x1="-45.72" y1="-33.02" x2="-45.72" y2="-35.56" width="0.1524" layer="91"/>
+<wire x1="-45.72" y1="-33.02" x2="-40.64" y2="-33.02" width="0.1524" layer="91"/>
+<junction x="-45.72" y="-33.02"/>
+<wire x1="-40.64" y1="-33.02" x2="-40.64" y2="-38.1" width="0.1524" layer="91"/>
+<pinref part="U1" gate="G$1" pin="XIN"/>
+<wire x1="-40.64" y1="-38.1" x2="-25.4" y2="-38.1" width="0.1524" layer="91"/>
+</segment>
+</net>
+<net name="N$12" class="0">
+<segment>
+<pinref part="C15" gate="G$1" pin="2"/>
+<pinref part="Q1" gate="G$1" pin="1"/>
+<wire x1="-48.26" y1="-43.18" x2="-45.72" y2="-43.18" width="0.1524" layer="91"/>
+<wire x1="-45.72" y1="-43.18" x2="-45.72" y2="-40.64" width="0.1524" layer="91"/>
+<wire x1="-45.72" y1="-43.18" x2="-40.64" y2="-43.18" width="0.1524" layer="91"/>
+<wire x1="-40.64" y1="-43.18" x2="-40.64" y2="-40.64" width="0.1524" layer="91"/>
+<junction x="-45.72" y="-43.18"/>
+<pinref part="R45" gate="G$1" pin="2"/>
+<wire x1="-40.64" y1="-40.64" x2="-38.1" y2="-40.64" width="0.1524" layer="91"/>
+</segment>
+</net>
+<net name="N$15" class="0">
+<segment>
+<pinref part="U1" gate="G$1" pin="XOUT"/>
+<pinref part="R45" gate="G$1" pin="1"/>
+<wire x1="-25.4" y1="-40.64" x2="-27.94" y2="-40.64" width="0.1524" layer="91"/>
+</segment>
+</net>
+<net name="VCC" class="0">
+<segment>
+<pinref part="C16" gate="G$1" pin="2"/>
+<wire x1="152.4" y1="-33.02" x2="170.18" y2="-33.02" width="0.1524" layer="91"/>
+<wire x1="170.18" y1="-33.02" x2="170.18" y2="-17.78" width="0.1524" layer="91"/>
+<pinref part="IC9" gate="G$1" pin="VCC"/>
+<wire x1="170.18" y1="-17.78" x2="165.1" y2="-17.78" width="0.1524" layer="91"/>
+<pinref part="P+12" gate="VCC" pin="VCC"/>
+<wire x1="170.18" y1="-2.54" x2="170.18" y2="-17.78" width="0.1524" layer="91"/>
+<junction x="170.18" y="-17.78"/>
+</segment>
+<segment>
+<pinref part="P+15" gate="VCC" pin="VCC"/>
+<pinref part="R46" gate="G$1" pin="1"/>
+<wire x1="129.54" y1="2.54" x2="129.54" y2="0" width="0.1524" layer="91"/>
+</segment>
+</net>
+<net name="QSPI_SD3" class="0">
+<segment>
+<pinref part="IC9" gate="G$1" pin="RES#/IO3"/>
+<wire x1="165.1" y1="-20.32" x2="172.72" y2="-20.32" width="0.1524" layer="91"/>
+<label x="172.72" y="-20.32" size="1.778" layer="95"/>
+</segment>
+<segment>
+<pinref part="U1" gate="G$1" pin="QSPI_SD3"/>
+<wire x1="20.32" y1="-33.02" x2="35.56" y2="-33.02" width="0.1524" layer="91"/>
+<label x="35.56" y="-33.02" size="1.778" layer="95"/>
+</segment>
+</net>
+<net name="QSPI_SCLK" class="0">
+<segment>
+<pinref part="IC9" gate="G$1" pin="CLK"/>
+<wire x1="165.1" y1="-22.86" x2="172.72" y2="-22.86" width="0.1524" layer="91"/>
+<label x="172.72" y="-22.86" size="1.778" layer="95"/>
+</segment>
+<segment>
+<pinref part="U1" gate="G$1" pin="QSPI_SCLK"/>
+<wire x1="20.32" y1="-22.86" x2="35.56" y2="-22.86" width="0.1524" layer="91"/>
+<label x="35.56" y="-22.86" size="1.778" layer="95"/>
+</segment>
+</net>
+<net name="QSPI_SD0" class="0">
+<segment>
+<pinref part="IC9" gate="G$1" pin="DIO/IO0"/>
+<wire x1="165.1" y1="-25.4" x2="172.72" y2="-25.4" width="0.1524" layer="91"/>
+<label x="172.72" y="-25.4" size="1.778" layer="95"/>
+</segment>
+<segment>
+<pinref part="U1" gate="G$1" pin="QSPI_SD0"/>
+<wire x1="20.32" y1="-25.4" x2="35.56" y2="-25.4" width="0.1524" layer="91"/>
+<label x="35.56" y="-25.4" size="1.778" layer="95"/>
+</segment>
+</net>
+<net name="QSPI_CSN" class="0">
+<segment>
+<pinref part="IC9" gate="G$1" pin="CS#"/>
+<wire x1="132.08" y1="-17.78" x2="129.54" y2="-17.78" width="0.1524" layer="91"/>
+<pinref part="R46" gate="G$1" pin="2"/>
+<wire x1="129.54" y1="-17.78" x2="124.46" y2="-17.78" width="0.1524" layer="91"/>
+<wire x1="129.54" y1="-10.16" x2="129.54" y2="-12.7" width="0.1524" layer="91"/>
+<junction x="129.54" y="-17.78"/>
+<label x="111.76" y="-17.78" size="1.778" layer="95"/>
+<pinref part="R47" gate="G$1" pin="2"/>
+<wire x1="129.54" y1="-12.7" x2="129.54" y2="-17.78" width="0.1524" layer="91"/>
+<wire x1="124.46" y1="-12.7" x2="129.54" y2="-12.7" width="0.1524" layer="91"/>
+<junction x="129.54" y="-12.7"/>
+</segment>
+<segment>
+<pinref part="U1" gate="G$1" pin="QSPI_CSN"/>
+<wire x1="20.32" y1="-35.56" x2="35.56" y2="-35.56" width="0.1524" layer="91"/>
+<label x="35.56" y="-35.56" size="1.778" layer="95"/>
+</segment>
+</net>
+<net name="QSPI_SD1" class="0">
+<segment>
+<pinref part="IC9" gate="G$1" pin="DO/IO1"/>
+<wire x1="132.08" y1="-20.32" x2="124.46" y2="-20.32" width="0.1524" layer="91"/>
+<label x="111.76" y="-20.32" size="1.778" layer="95"/>
+</segment>
+<segment>
+<pinref part="U1" gate="G$1" pin="QSPI_SD1"/>
+<wire x1="20.32" y1="-27.94" x2="35.56" y2="-27.94" width="0.1524" layer="91"/>
+<label x="35.56" y="-27.94" size="1.778" layer="95"/>
+</segment>
+</net>
+<net name="QSPI_SD2" class="0">
+<segment>
+<pinref part="IC9" gate="G$1" pin="WP#/IO2"/>
+<wire x1="132.08" y1="-22.86" x2="124.46" y2="-22.86" width="0.1524" layer="91"/>
+<label x="111.76" y="-22.86" size="1.778" layer="95"/>
+</segment>
+<segment>
+<pinref part="U1" gate="G$1" pin="QSPI_SD2"/>
+<wire x1="20.32" y1="-30.48" x2="35.56" y2="-30.48" width="0.1524" layer="91"/>
+<label x="35.56" y="-30.48" size="1.778" layer="95"/>
+</segment>
+</net>

Commit message: ASAS
Parts:
- removed U1: RP2040, RP2040:RP2040
- added C17, C18, C19, C20, C21, C22, C23, C26, C27: (no value), rcl:C-EUC0805
- added C24, C25: 1u, rcl:C-EUC0805
- added U$1: RP2040, jason_eagle6:RP2040
Connections:
- new net +1V1: C25.2, C26.2, C27.2, U$1.DVDD1, U$1.DVDD2, U$1.VREG_VOUT
- new net +3V3: C17.2, C18.2, C19.2, C20.2, C21.2, C22.2, C23.2, C24.2, U$1.ADC_AVDD, U$1.IOVDD1, U$1.IOVDD2, U$1.IOVDD3, U$1.IOVDD4, U$1.IOVDD5, U$1.IOVDD6, U$1.USB_VDD, U$1.VREG_VIN
- new net N$44: U$1.TESTEN
- new net N$45: U$1.SWCLK
- new net N$46: U$1.SWDIO
- new net N$47: U$1.RUN
- new net N$65: U$1.GPIO25
- new net USB_DM: U$1.USB_DM
- new net USB_DP: U$1.USB_DP
- net AUXIN: now also U$1.GPIO19
- net AUXOUT: now also U$1.GPIO18
- net D_ADT: now also U$1.GPIO15
- net D_ARK: now also U$1.GPIO13
- net D_ENA: now also U$1.GPIO22
- net D_KCK: now also U$1.GPIO12, U$1.GPIO14
- net D_KDT: now also U$1.GPIO11
- net ENC1: now also U$1.GPIO0
- net ENC2: now also U$1.GPIO1
- net GATE1: now also U$1.GPIO7
- net GATE2: now also U$1.GPIO8
- net GATE3: now also U$1.GPIO9
- net GATE4: now also U$1.GPIO10
- net GND: now also C17.1, C18.1, C19.1, C20.1, C21.1, C22.1, C23.1, C24.1, C25.1, C26.1, C27.1, U$1.GND; no longer U1.GND
- net I2C0SCL: now also U$1.GPIO21
- net I2C0SDA: now also U$1.GPIO20
- net I2C1SCL: now also U$1.GPIO27/ADC1
- net I2C1SDA: now also U$1.GPIO26/ADC0
- net KEY_READ1: now also U$1.GPIO28/ADC2
- net KEY_READ2: now also U$1.GPIO29/ADC3
- net LED1: now also U$1.GPIO4
- net LED2: now also U$1.GPIO5
- net LED3: now also U$1.GPIO6
- net MIDIRX: now also U$1.GPIO17
- net MIDITX: now also U$1.GPIO16
- net N$10: now also U$1.XIN; no longer U1.XIN
- net N$15: now also U$1.XOUT; no longer U1.XOUT
- net OFF_SW: now also U$1.GPIO2
- net PWR_CTRL: now also U$1.GPIO3
- net QSPI_CSN: now also U$1.QSPI_SS#; no longer U1.QSPI_CSN
- net QSPI_SCLK: now also U$1.QSPI_SCLK; no longer U1.QSPI_SCLK
- net QSPI_SD0: now also U$1.QSPI_SD0; no longer U1.QSPI_SD0
- net QSPI_SD1: now also U$1.QSPI_SD1; no longer U1.QSPI_SD1
- net QSPI_SD2: now also U$1.QSPI_SD2; no longer U1.QSPI_SD2
- net QSPI_SD3: now also U$1.QSPI_SD3; no longer U1.QSPI_SD3
- net SYNCIN: now also U$1.GPIO23
- net SYNCOUT: now also U$1.GPIO24
Other:
- moved on the sheet: C14, C15, Q1, R45
