File: matrix_main_board.sch (EAGLE design)
At the start: 124 parts, among them IC1 MKE02_44PIN, IC2 24AA01SM, IC3 74HC595D, IC4 74HC595D, IC5 74HC595D, IC6 74HC595D, IC7 NPIC6C596, IC8 NPIC6C596

Commit message: VERSION 1
Other:
- note added: "DISPLAY MATRIX AND DRIVERS"
- note added: "EEPROM"
- note added: "MATRIX SEQUENCER MAIN/DISPLAY BOARD"
- note added: "MCU"
- note added: "SWITCH MATRIX"
- note added: "Version 1 - 10 July 2018 - J Hotchkiss / Sixty Four Pixels"
- moved on the sheet: C1, C11, C12, C13, C2, C3, C4, CKOUT, CLKIN, ENC1, ENC2, G1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

Commit message: values
Parts:
- C11, C2: value (none) -> 18p
- R1, R2: value (none) -> 4k7
- XTL1: value (none) -> 20m
Changed lines of the file:
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@@
 <part name="P+8" library="supply1" deviceset="+5V" device=""/>
 <part name="IC1" library="jason_eagle6" deviceset="MKE02_44PIN" device=""/>
-<part name="XTL1" library="crystal" deviceset="CRYSTAL" device="HC49S"/>
-<part name="C2" library="rcl" deviceset="C-EU" device="C0805"/>
-<part name="C11" library="rcl" deviceset="C-EU" device="C0805"/>
+<part name="XTL1" library="crystal" deviceset="CRYSTAL" device="HC49S" value="20m"/>
+<part name="C2" library="rcl" deviceset="C-EU" device="C0805" value="18p"/>
+<part name="C11" library="rcl" deviceset="C-EU" device="C0805" value="18p"/>
 <part name="R6" library="rcl" deviceset="R-EU_" device="R0805"/>
 <part name="GND6" library="supply1" deviceset="GND" device=""/>
@@
 <part name="C3" library="rcl" deviceset="C-EU" device="C0805"/>
 <part name="GND12" library="supply1" deviceset="GND" device=""/>
-<part name="R2" library="rcl" deviceset="R-EU_" device="R0805"/>
-<part name="R1" library="rcl" deviceset="R-EU_" device="R0805"/>
+<part name="R2" library="rcl" deviceset="R-EU_" device="R0805" value="4k7"/>
+<part name="R1" library="rcl" deviceset="R-EU_" device="R0805" value="4k7"/>
 <part name="P+11" library="supply1" deviceset="+5V" device=""/>
 <part name="P+12" library="supply1" deviceset="+5V" device=""/>

Commit message: changes for rev2
Parts:
- removed ENC2, GND: (no value), pinhead:PINHD-1X1
- removed PB4: TPTP17R, testpad:TPTP17R
- added D10, D11, D9: 0805DIODE, jasons_stuff:0805DIODE
- added SW10, SW11, SW9: (no value), switch-omron:10-XX
- ENC1: value (none) -> ENCODER; device pinhead:PINHD-1X1 -> jason_eagle6:ENCODER
Connections:
- net KEY_READ renamed KEY_READ1
- removed net PTB4: IC1.PTB4, PB4.TP
- new net KEY_READ2: IC1.PTB4, SW10.P1, SW11.P1, SW9.P1
- new net N$1: D10.P$1, SW10.S
- new net N$7: D9.P$1, SW11.S
- new net N$8: D11.P$1, SW9.S
- net ENC1: now also ENC1.B; no longer ENC1.1
- net ENC2: now also ENC1.A; no longer ENC2.1
- net GND: now also ENC1.C; no longer GND.1
- net K13: now also D11.P$2
- net K14: now also D10.P$2
- net K15: now also D9.P$2
Other:
- note added: "Version 2 - 19 MAY 19 - J Hotchkiss / Sixty Four Pixels"
- note removed: "Version 1 - 10 July 2018 - J Hotchkiss / Sixty Four Pixels"
Changed lines of the file:
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@@
 <layer number="56" name="wert" color="7" fill="1" visible="no" active="no"/>
 <layer number="57" name="tCAD" color="7" fill="1" visible="no" active="no"/>
+<layer number="90" name="Modules" color="7" fill="1" visible="yes" active="yes"/>
 <layer number="91" name="Nets" color="2" fill="1" visible="yes" active="yes"/>
 <layer number="92" name="Busses" color="1" fill="1" visible="yes" active="yes"/>
@@
 <part name="OFFSW" library="pinhead" deviceset="PINHD-1X1" device=""/>
 <part name="PWRCTL" library="pinhead" deviceset="PINHD-1X1" device=""/>
-<part name="ENC1" library="pinhead" deviceset="PINHD-1X1" device=""/>
-<part name="ENC2" library="pinhead" deviceset="PINHD-1X1" device=""/>
 <part name="SWD_CLK" library="pinhead" deviceset="PINHD-1X1" device=""/>
 <part name="RESET" library="pinhead" deviceset="PINHD-1X1" device=""/>
@@
 <part name="PE0" library="testpad" deviceset="TP" device="TP17R"/>
 <part name="PC7" library="testpad" deviceset="TP" device="TP17R"/>
-<part name="PB4" library="testpad" deviceset="TP" device="TP17R"/>
 <part name="PD7" library="testpad" deviceset="TP" device="TP17R"/>
 <part name="PD6" library="testpad" deviceset="TP" device="TP17R"/>
@@
 <part name="GD1" library="pinhead" deviceset="PINHD-1X1" device=""/>
 <part name="GD2" library="pinhead" deviceset="PINHD-1X1" device=""/>
-<part name="GND" library="pinhead" deviceset="PINHD-1X1" device=""/>
 <part name="GND17" library="supply1" deviceset="GND" device=""/>
 <part name="VCC2" library="pinhead" deviceset="PINHD-1X1" device=""/>
@@
 <part name="GND19" library="supply1" deviceset="GND" device=""/>
 <part name="C13" library="rcl" deviceset="CPOL-EU" device="E2.5-7"/>
+<part name="ENC1" library="jason_eagle6" deviceset="ENCODER" device=""/>
+<part name="SW11" library="switch-omron" deviceset="10-XX" device=""/>
+<part name="SW10" library="switch-omron" deviceset="10-XX" device=""/>
+<part name="SW9" library="switch-omron" deviceset="10-XX" device=""/>
+<part name="D9" library="jasons_stuff" deviceset="0805DIODE" device=""/>
+<part name="D10" library="jasons_stuff" deviceset="0805DIODE" device=""/>
+<part name="D11" library="jasons_stuff" deviceset="0805DIODE" device=""/>
 </parts>
 <sheets>
@@
 <text x="48.26" y="190.5" size="10.16" layer="97">EEPROM</text>
 <text x="114.3" y="27.94" size="10.16" layer="97">MATRIX SEQUENCER MAIN/DISPLAY BOARD</text>
-<text x="114.3" y="12.7" size="10.16" layer="97">Version 1 - 10 July 2018 - J Hotchkiss / Sixty Four Pixels</text>
+<text x="114.3" y="12.7" size="10.16" layer="97">Version 2 - 19 MAY 19 - J Hotchkiss / Sixty Four Pixels</text>
 </plain>
 <instances>
@@
 <instance part="OFFSW" gate="G$1" x="266.7" y="91.44" rot="R90"/>
 <instance part="PWRCTL" gate="G$1" x="274.32" y="91.44" rot="R90"/>
-<instance part="ENC1" gate="G$1" x="289.56" y="91.44" rot="R90"/>
-<instance part="ENC2" gate="G$1" x="297.18" y="91.44" rot="R90"/>
 <instance part="SWD_CLK" gate="G$1" x="-45.72" y="152.4" rot="R180"/>
 <instance part="RESET" gate="G$1" x="-45.72" y="144.78" rot="R180"/>
@@
 <instance part="PE0" gate="G$1" x="-15.24" y="142.24"/>
 <instance part="PC7" gate="G$1" x="-5.08" y="142.24"/>
-<instance part="PB4" gate="G$1" x="-22.86" y="48.26" rot="R180"/>
 <instance part="PD7" gate="G$1" x="-15.24" y="48.26" rot="R180"/>
 <instance part="PD6" gate="G$1" x="-12.7" y="48.26" rot="R180"/>
@@
 <attribute name="VALUE" x="176.53" y="137.16" size="1.778" layer="96" rot="R180"/>
 </instance>
-<instance part="GND" gate="G$1" x="304.8" y="91.44" smashed="yes" rot="R90">
-<attribute name="NAME" x="301.625" y="85.09" size="1.778" layer="95" rot="R90"/>
-<attribute name="VALUE" x="309.88" y="85.09" size="1.778" layer="96" rot="R90"/>
-</instance>
-<instance part="GND17" gate="1" x="312.42" y="78.74" rot="R90"/>
+<instance part="GND17" gate="1" x="274.32" y="149.86"/>
 <instance part="VCC2" gate="G$1" x="-45.72" y="170.18" smashed="yes" rot="R180">
 <attribute name="NAME" x="-39.37" y="167.005" size="1.778" layer="95" rot="R180"/>
@@
 <instance part="GND19" gate="1" x="-33.02" y="157.48"/>
 <instance part="C13" gate="G$1" x="190.5" y="152.4"/>
+<instance part="ENC1" gate="G$1" x="271.78" y="167.64"/>
+<instance part="SW11" gate="1" x="462.28" y="287.02" rot="R180"/>
+<instance part="SW10" gate="1" x="449.58" y="287.02" rot="R180"/>
+<instance part="SW9" gate="1" x="436.88" y="287.02" rot="R180"/>
+<instance part="D9" gate="G$1" x="462.28" y="274.32" rot="R180"/>
+<instance part="D10" gate="G$1" x="449.58" y="274.32" rot="R180"/>
+<instance part="D11" gate="G$1" x="436.88" y="274.32" rot="R180"/>
 </instances>
 <busses>
@@
 <junction x="22.86" y="292.1"/>
 <junction x="-33.02" y="236.22"/>
+<pinref part="D11" gate="G$1" pin="P$2"/>
+<wire x1="436.88" y1="254" x2="436.88" y2="273.812" width="0.1524" layer="91"/>
+<wire x1="396.24" y1="254" x2="436.88" y2="254" width="0.1524" layer="91"/>
+<junction x="396.24" y="254"/>
 </segment>
 </net>
@@
 <junction x="289.56" y="284.48"/>
 <junction x="-33.02" y="238.76"/>
+<pinref part="D10" gate="G$1" pin="P$2"/>
+<wire x1="449.58" y1="251.46" x2="449.58" y2="273.812" width="0.1524" layer="91"/>
+<wire x1="403.86" y1="251.46" x2="449.58" y2="251.46" width="0.1524" layer="91"/>
+<junction x="403.86" y="251.46"/>
 </segment>
 </net>
@@
 <junction x="289.56" y="276.86"/>
 <junction x="-33.02" y="241.3"/>
+<pinref part="D9" gate="G$1" pin="P$2"/>
+<wire x1="462.28" y1="248.92" x2="462.28" y2="273.812" width="0.1524" layer="91"/>
+<wire x1="411.48" y1="248.92" x2="462.28" y2="248.92" width="0.1524" layer="91"/>
+<junction x="411.48" y="248.92"/>
 </segment>
 </net>
@@
 </segment>
 <segment>
-<pinref part="GND" gate="G$1" pin="1"/>
 <pinref part="GND17" gate="1" pin="GND"/>
-<wire x1="304.8" y1="88.9" x2="304.8" y2="78.74" width="0.1524" layer="91"/>
-<wire x1="304.8" y1="78.74" x2="309.88" y2="78.74" width="0.1524" layer="91"/>
+<wire x1="274.32" y1="152.4" x2="274.32" y2="160.02" width="0.1524" layer="91"/>
+<pinref part="ENC1" gate="G$1" pin="C"/>
 </segment>
 <segment>
@@
 </segment>
 <segment>
-<pinref part="ENC1" gate="G$1" pin="1"/>
-<wire x1="289.56" y1="88.9" x2="289.56" y2="68.58" width="0.1524" layer="91"/>
-<label x="289.56" y="68.58" size="1.778" layer="95" rot="R90"/>
+<wire x1="271.78" y1="160.02" x2="271.78" y2="157.48" width="0.1524" layer="91"/>
+<label x="271.78" y="152.4" size="1.778" layer="95" rot="R90"/>
+<pinref part="ENC1" gate="G$1" pin="B"/>
 </segment>
 </net>
@@
 </segment>
 <segment>
-<pinref part="ENC2" gate="G$1" pin="1"/>
-<wire x1="297.18" y1="88.9" x2="297.18" y2="71.12" width="0.1524" layer="91"/>
-<label x="297.18" y="68.58" size="1.778" layer="95" rot="R90"/>
+<wire x1="269.24" y1="160.02" x2="269.24" y2="157.48" width="0.1524" layer="91"/>
+<label x="269.24" y="152.4" size="1.778" layer="95" rot="R90"/>
+<pinref part="ENC1" gate="G$1" pin="A"/>
 </segment>
 </net>
@@
 <wire x1="233.68" y1="160.02" x2="233.68" y2="170.18" width="0.1524" layer="91"/>
 <label x="233.68" y="170.18" size="1.778" layer="95" rot="R90"/>
-</segment>
-</net>
-<net name="PTB4" class="0">
-<segment>
-<pinref part="IC1" gate="G$1" pin="PTB4"/>
-<wire x1="-22.86" y1="71.12" x2="-22.86" y2="50.8" width="0.1524" layer="91"/>
-<label x="-22.86" y="55.88" size="1.778" layer="95" rot="R90"/>
-<pinref part="PB4" gate="G$1" pin="TP"/>
 </segment>
 </net>
@@
 </segment>
 </net>
-<net name="KEY_READ" class="0">
+<net name="KEY_READ1" class="0">
 <segment>
 <pinref part="IC1" gate="G$1" pin="PTC6"/>
@@
 </segment>
 </net>
+<net name="N$8" class="0">
+<segment>
+<pinref part="D11" gate="G$1" pin="P$1"/>
+<pinref part="SW9" gate="1" pin="S"/>
+<wire x1="436.88" y1="278.892" x2="436.88" y2="281.94" width="0.1524" layer="91"/>
+</segment>
+</net>
+<net name="KEY_READ2" class="0">
+<segment>
+<wire x1="434.34" y1="297.18" x2="447.04" y2="297.18" width="0.1524" layer="91"/>
+<label x="472.44" y="297.18" size="1.778" layer="95"/>
+<pinref part="SW9" gate="1" pin="P1"/>
+<wire x1="447.04" y1="297.18" x2="459.74" y2="297.18" width="0.1524" layer="91"/>
+<wire x1="459.74" y1="297.18" x2="472.44" y2="297.18" width="0.1524" layer="91"/>
+<wire x1="434.34" y1="297.18" x2="434.34" y2="292.1" width="0.1524" layer="91"/>
+<pinref part="SW10" gate="1" pin="P1"/>
+<wire x1="447.04" y1="292.1" x2="447.04" y2="297.18" width="0.1524" layer="91"/>
+<junction x="447.04" y="297.18"/>
+<pinref part="SW11" gate="1" pin="P1"/>
+<wire x1="459.74" y1="292.1" x2="459.74" y2="297.18" width="0.1524" layer="91"/>
+<junction x="459.74" y="297.18"/>
+</segment>
+<segment>
+<pinref part="IC1" gate="G$1" pin="PTB4"/>
+<wire x1="-22.86" y1="71.12" x2="-22.86" y2="55.88" width="0.1524" layer="91"/>
+<label x="-22.86" y="55.88" size="1.778" layer="95" rot="R90"/>
+</segment>
+</net>
+<net name="N$1" class="0">
+<segment>
+<pinref part="D10" gate="G$1" pin="P$1"/>
+<pinref part="SW10" gate="1" pin="S"/>
+<wire x1="449.58" y1="278.892" x2="449.58" y2="281.94" width="0.1524" layer="91"/>
+</segment>
+</net>
+<net name="N$7" class="0">
+<segment>
+<pinref part="D9" gate="G$1" pin="P$1"/>
+<pinref part="SW11" gate="1" pin="S"/>
+<wire x1="462.28" y1="278.892" x2="462.28" y2="281.94" width="0.1524" layer="91"/>
+</segment>
+</net>

Commit message: works in progress
Parts:
- removed PC7, PE0, PE7: TPTP17R, testpad:TPTP17R
- added AUXIN, GD5: (no value), pinhead:PINHD-1X1
- added R43, R44: 4k7, rcl:R-EU_R0805
- DISP1, DISP2, DISP3, DISP4, DISP5, DISP6, DISP7, DISP8: value 1388BBMATRIX -> 1388BBMATRIX24PIN; device jason_eagle6:1388BBMATRIX -> jason_eagle6:1388BBMATRIX24PIN
Connections:
- net AUXGATE renamed AUXOUT
- removed net I2CSCL: IC1.PTA3, IC2.SCL, R2.1, SCL.1
- removed net I2CSDA: IC1.PTA2, IC2.SDA, R1.1, SDA.1
- removed net PTC7: IC1.PTC7, PC7.TP
- removed net PTE0: IC1.PTE0, PE0.TP
- removed net PTE7: IC1.PTE7, PE7.TP
- new net AUXIN: AUXIN.1, IC1.PTC7
- new net I2C0SCL: IC1.PTA3, R43.1, SCL.1
- new net I2C0SDA: IC1.PTA2, R44.1, SDA.1
- new net I2C1SCL: IC1.PTE1, IC2.SCL, R1.1
- new net I2C1SDA: IC1.PTE0, IC2.SDA, R2.1
- net +5V: now also R43.2, R44.2
- net GND: now also GD5.1
- net OFF_SW: now also IC1.PTE7; no longer IC1.PTE1
Other:
- moved on the sheet: R1, R2

Commit message: V3 candidate
Other:
- note added: "NOODLEBOX MAIN/DISPLAY BOARD"
- note added: "Version 3 - 26 NOV 19 - J Hotchkiss / Sixty Four Pixels"
- note removed: "MATRIX SEQUENCER MAIN/DISPLAY BOARD"
- note removed: "Version 2 - 19 MAY 19 - J Hotchkiss / Sixty Four Pixels"
Changed lines of the file:
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@@
 <text x="-33.02" y="25.4" size="10.16" layer="97">MCU</text>
 <text x="48.26" y="190.5" size="10.16" layer="97">EEPROM</text>
-<text x="114.3" y="27.94" size="10.16" layer="97">MATRIX SEQUENCER MAIN/DISPLAY BOARD</text>
-<text x="114.3" y="12.7" size="10.16" layer="97">Version 2 - 19 MAY 19 - J Hotchkiss / Sixty Four Pixels</text>
+<text x="114.3" y="27.94" size="10.16" layer="97">NOODLEBOX MAIN/DISPLAY BOARD</text>
+<text x="114.3" y="12.7" size="10.16" layer="97">Version 3 - 26 NOV 19 - J Hotchkiss / Sixty Four Pixels</text>
 </plain>
 <instances>

Commit message: in prog
Parts:
- added U$1: MKE02_64PIN64, jason_eagle6:MKE02_64PIN64
Connections:
- removed net PTD6: IC1.PTD6, PD6.TP
- removed net PTD7: IC1.PTD7, PD7.TP
- new net N$10: PD7.TP, U$1.PTD7
- new net N$12: PD6.TP, U$1.PTD6
- net +5V: now also U$1.VDD, U$1.VDD1, U$1.VDDA/REFH
- net AUXIN: now also U$1.PTC7
- net AUXOUT: now also U$1.PTA7
- net D_ACK: now also U$1.PTB2
- net D_ADT: now also U$1.PTB3
- net D_ARK: now also U$1.PTC0
- net D_ENA: now also U$1.PTA1
- net D_KCK: now also U$1.PTC1
- net D_KDT: now also U$1.PTD5
- net ENC1: now also U$1.PTD1
- net ENC2: now also U$1.PTD0
- net GATE1: now also U$1.PTD2
- net GATE2: now also U$1.PTD3
- net GATE3: now also U$1.PTD4
- net GATE4: now also U$1.PTA6
- net GND: now also U$1.VSS, U$1.VSS1, U$1.VSSA/VSS
- net I2C0SCL: now also U$1.PTA3
- net I2C0SDA: now also U$1.PTA2
- net I2C1SCL: now also U$1.PTE1
- net I2C1SDA: now also U$1.PTE0
- net KEY_READ1: now also U$1.PTC6
- net KEY_READ2: now also U$1.PTB4
- net LED1: now also U$1.PTB5
- net LED2: now also U$1.PTC3
- net LED3: now also U$1.PTC2
- net MIDIRX: now also U$1.PTB0
- net MIDITX: now also U$1.PTB1
- net N$4: now also U$1.PTB7; no longer IC1.PTB7
- net N$5: now also U$1.PTB6; no longer IC1.PTB6
- net NRESET: now also U$1.PTA5; no longer IC1.PTA5
- net OFF_SW: now also U$1.PTE7
- net PTH2: now also U$1.PTH2; no longer IC1.PTH2
- net PWR_CTRL: now also U$1.PTE2
- net SWDCLK: now also U$1.PTC4; no longer IC1.PTC4
- net SWDIO: now also U$1.PTA4; no longer IC1.PTA4
- net SYNCIN: now also U$1.PTA0
- net SYNCOUT: now also U$1.PTC5
Other:
- moved on the sheet: C1, C11, C2, C4, GD4, PD6, PD7, PH2, R3, R4, R5, R6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

Commit message: work in prog
Parts:
- removed IC1: MKE02_44PIN, jason_eagle6:MKE02_44PIN
Connections:
- net +5V: no longer IC1.VDD, IC1.VDD1, IC1.VDDA/REFH
- net AUXIN: no longer IC1.PTC7
- net AUXOUT: no longer IC1.PTA7
- net D_ACK: no longer IC1.PTB2
- net D_ADT: no longer IC1.PTB3
- net D_ARK: no longer IC1.PTC0
- net D_ENA: no longer IC1.PTA1
- net D_KCK: no longer IC1.PTC1
- net D_KDT: no longer IC1.PTD5
- net ENC1: no longer IC1.PTD1
- net ENC2: no longer IC1.PTD0
- net GATE1: no longer IC1.PTD2
- net GATE2: no longer IC1.PTD3
- net GATE3: no longer IC1.PTD4
- net GATE4: no longer IC1.PTA6
- net GND: no longer IC1.VSS, IC1.VSS1, IC1.VSSA/VSS
- net I2C0SCL: no longer IC1.PTA3
- net I2C0SDA: no longer IC1.PTA2
- net I2C1SCL: no longer IC1.PTE1
- net I2C1SDA: no longer IC1.PTE0
- net KEY_READ1: no longer IC1.PTC6
- net KEY_READ2: no longer IC1.PTB4
- net LED1: no longer IC1.PTB5
- net LED2: no longer IC1.PTC3
- net LED3: no longer IC1.PTC2
- net MIDIRX: no longer IC1.PTB0
- net MIDITX: no longer IC1.PTB1
- net OFF_SW: no longer IC1.PTE7
- net PWR_CTRL: no longer IC1.PTE2
- net SYNCIN: no longer IC1.PTA0
- net SYNCOUT: no longer IC1.PTC5
Other:
- note added: "Version 4 - 30 JUL 22 - J Hotchkiss / Sixty Four Pixels"
- note removed: "Version 3 - 26 NOV 19 - J Hotchkiss / Sixty Four Pixels"
- moved on the sheet: C1, C11, C2, C4, GD4, PD6, PD7, PH2, R3, R4, R5, R6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

Commit message: 64pin
Parts:
- removed R3, R4, R5: (no value), rcl:R-EU_R0805
- added PE6, PF4, PF5, PF6, PF7, PG0, PG1, PG2, PH0, PH1, PH6, PH7: TPTP17R, testpad:TPTP17R
- renumbered GD4 to GD, RESET to RT, SWD_CLK to CK, SWD_DAT to DT, U$1 to IC1, VCC2 to VC
Connections:
- new net N$15: IC1.PTF7, PF7.TP
- new net N$25: IC1.PTF6, PF6.TP
- new net N$26: IC1.PTF5, PF5.TP
- new net N$27: IC1.PTF4, PF4.TP
- new net N$36: IC1.PTH1, PH1.TP
- new net N$37: IC1.PTH0, PH0.TP
- new net N$38: IC1.PTE6, PE6.TP
- new net N$41: IC1.PTH6, PH6.TP
- new net N$43: IC1.PTG1, PG1.TP
- new net PG0: IC1.PTG0, PG0.TP
- new net PTG2: IC1.PTG2, PG2.TP
- new net PTH7: IC1.PTH7, PH7.TP
- net +5V: no longer R3.2, R4.2, R5.2
- net NRESET: no longer R3.1
- net SWDCLK: no longer R5.1
- net SWDIO: no longer R4.1
