File: matrix_main_board.sch (EAGLE design)
At the start: 137 parts, among them IC1 MKE02_64PIN64, IC2 24AA01SM, IC3 74HC595D, IC4 74HC595D, IC5 74HC595D, IC6 74HC595D, IC7 NPIC6C596, IC8 NPIC6C596

Commit message: correct footprint
Parts:
- IC1: value MKE02_64PIN64 -> MKE02_64PINQFP64; device jason_eagle6:MKE02_64PIN64 -> jason_eagle6:MKE02_64PINQFP64
Changed lines of the file:
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@@
 <part name="R44" library="rcl" deviceset="R-EU_" device="R0805" value="4k7"/>
 <part name="P+14" library="supply1" deviceset="+5V" device=""/>
-<part name="IC1" library="jason_eagle6" deviceset="MKE02_64PIN" device="64"/>
+<part name="IC1" library="jason_eagle6" deviceset="MKE02_64PIN" device="QFP64" value="MKE02_64PINQFP64"/>
 <part name="GND14" library="supply1" deviceset="GND" device=""/>
 <part name="P+12" library="supply1" deviceset="+5V" device=""/>

Commit message: V5 BOARD
Other:
- note added: "CC-NC-BY-SA"
- note added: "Version 4 - NOV 22 - J Hotchkiss / Sixty Four Pixels"
- note removed: "Version 4 - 30 JUL 22 - J Hotchkiss / Sixty Four Pixels"
Changed lines of the file:
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@@
 <text x="48.26" y="190.5" size="10.16" layer="97">EEPROM</text>
 <text x="114.3" y="27.94" size="10.16" layer="97">NOODLEBOX MAIN/DISPLAY BOARD</text>
-<text x="114.3" y="12.7" size="10.16" layer="97">Version 4 - 30 JUL 22 - J Hotchkiss / Sixty Four Pixels</text>
+<text x="114.3" y="12.7" size="10.16" layer="97">Version 4 - NOV 22 - J Hotchkiss / Sixty Four Pixels</text>
+<text x="114.3" y="-2.032" size="10.16" layer="97">CC-NC-BY-SA</text>
 </plain>
 <instances>
