File: matrix_main_board.brd (EAGLE design)
At the start: 155.7 x 95.9 mm, 124 parts, among them IC1 MKE02_44PIN, IC2 24AA01SM, IC3 74HC595D, IC4 74HC595D, IC5 74HC595D, IC6 74HC595D, IC7 NPIC6C596, IC8 NPIC6C596

Commit message: values
Parts:
- C11, C2: value (none) -> 18p
- R1, R2: value (none) -> 4k7
- XTL1: value (none) -> 20m

Commit message: changes for rev2
Parts:
- removed ENC2, GND: (no value), pinhead:1X01
- removed PB4: TPTP17R, testpad:TP17R
- added D10, D11, D9: 0805DIODE, jasons_stuff:0805DIODE
- added SW10, SW11, SW9: (no value), switch-omron:B3F-10XX
- ENC1: value (none) -> ENCODER; device pinhead:1X01 -> jason_eagle6:ENCODER
- moved ENC1 19.2 mm to (144.8, 21.6), turned to 180 degrees
- moved C12 12.2 mm to (141.2, 35.6)
- moved C13 12.0 mm to (148.6, 35.6)
Connections:
- net KEY_READ renamed KEY_READ1
- removed net PTB4: IC1.13, PB4.TP
- new net KEY_READ2: IC1.13, SW10.4, SW11.4, SW9.4
- new net N$1: D10.C, SW10.1
- new net N$7: D9.C, SW11.1
- new net N$8: D11.C, SW9.1
- net ENC1: now also ENC1.B; no longer ENC1.1
- net ENC2: now also ENC1.A; no longer ENC2.1
- net GND: now also ENC1.C; no longer GND.1
- net K13: now also D11.A
- net K14: now also D10.A
- net K15: now also D9.A
Routing:
- net KEY_READ2: track 0.00 -> 47.2 mm
- net K14: track 147.0 -> 182.0 mm, vias 4 -> 6
- net ENC2: track 44.7 -> 79.6 mm
- net +5V: track 549.4 -> 515.1 mm
- net K13: track 156.5 -> 190.7 mm, vias 4 -> 6
- net K15: track 132.4 -> 165.5 mm
- net ENC1: track 43.2 -> 75.6 mm
- net PTB4: track 10.0 -> 0.00 mm
- net KEY_READ1: track 235.5 -> 245.2 mm, vias 3 -> 1
- net N$7: track 0.00 -> 3.03 mm
- net N$1: track 0.00 -> 3.03 mm
- net N$8: track 0.00 -> 3.03 mm
Other:
- board text added: "Matrix Sequencer Main Board v2"
- board text removed: "Matrix Sequencer Main Board v1"

Commit message: works in progress
Parts:
- removed PC7, PE0, PE7: TPTP17R, testpad:TP17R
- added AUXIN, GD5: (no value), pinhead:1X01
- added R43, R44: 4k7, rcl:R0805
- DISP1, DISP2, DISP3, DISP4, DISP5, DISP6, DISP7, DISP8: value 1388BBMATRIX -> 1388BBMATRIX24PIN; device jason_eagle6:1388LEDMATRIX -> jason_eagle6:1388_24PIN
- moved GD3 28.5 mm to (120.7, 91.9)
- moved R1 26.6 mm to (128.7, 76.8)
- moved R2 23.5 mm to (128.7, 79.4)
- moved VCC 20.6 mm to (125.7, 94.5)
- moved VCC1 18.8 mm to (125.7, 91.9)
- moved RX 13.2 mm to (128.3, 94.5)
- moved GD1 13.2 mm to (123.2, 94.5)
- moved TX 11.8 mm to (128.3, 91.9)
- moved GX 11.8 mm to (130.8, 91.9)
- moved G4 9.68 mm to (133.3, 91.9)
- moved G1 8.36 mm to (130.8, 94.5)
- moved GD2 8.36 mm to (120.7, 94.5)
- moved G3 7.84 mm to (135.9, 91.9)
- moved CKOUT 6.49 mm to (143.5, 91.9)
- moved SDA 6.49 mm to (138.4, 91.9)
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Connections:
- net AUXGATE renamed AUXOUT
- removed net I2CSCL: IC1.32, IC2.6, R2.1, SCL.1
- removed net I2CSDA: IC1.33, IC2.5, R1.1, SDA.1
- removed net PTC7: IC1.36, PC7.TP
- removed net PTE0: IC1.40, PE0.TP
- removed net PTE7: IC1.3, PE7.TP
- new net AUXIN: AUXIN.1, IC1.36
- new net I2C0SCL: IC1.32, R43.1, SCL.1
- new net I2C0SDA: IC1.33, R44.1, SDA.1
- new net I2C1SCL: IC1.39, IC2.6, R1.1
- new net I2C1SDA: IC1.40, IC2.5, R2.1
- net +5V: now also R43.2, R44.2
- net GND: now also GD5.1
- net OFF_SW: now also IC1.3; no longer IC1.39
Routing:
- net I2CSCL: track 56.3 -> 0.00 mm, vias 3 -> 0
- net I2CSDA: track 53.5 -> 0.00 mm, vias 3 -> 0
- net I2C1SDA: track 0.00 -> 39.3 mm, vias 0 -> 2
- net I2C1SCL: track 0.00 -> 34.7 mm, vias 0 -> 2
- net I2C0SCL: track 0.00 -> 24.9 mm, vias 0 -> 1
- net I2C0SDA: track 0.00 -> 18.0 mm, vias 0 -> 1
- net MIDITX: track 30.5 -> 15.3 mm, vias 1 -> 0
- net OFF_SW: track 17.4 -> 32.5 mm, vias 0 -> 2
- net AUXOUT: track 27.4 -> 13.2 mm
- net D_KDT: track 139.5 -> 125.6 mm, vias 3 -> 2
- net MIDIRX: track 30.6 -> 17.6 mm
- net AUXIN: track 0.00 -> 10.8 mm
- net SYNCOUT: track 22.5 -> 13.3 mm
- net GATE4: track 24.3 -> 15.4 mm
- net K8: track 194.8 -> 186.2 mm
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Other:
- board size 155.7 x 95.9 mm -> 155.7 x 92.3 mm
- board text added: "NOODLEBOX Main Board v3"
- board text removed: "Matrix Sequencer Main Board v2"

Commit message: dsfdfs
Parts:
- added C14, C15, C16: 18p, rcl:C0805
- added IC9: W25Q128, jason_eagle6:SO08
- added Q1: (no value), adafruit:CTS406
- added R45, R46, R47: (no value), rcl:R0805
- added U1: RP2040, RP2040:QFN40P700X700X90-57N
Connections:
- new net ADC_AVDD: U1.43
- new net DVDD: U1.23, U1.50
- new net IOVDD: U1.1, U1.10, U1.22, U1.33, U1.42, U1.49
- new net N$10: C14.2, Q1.3, U1.20
- new net N$12: C15.2, Q1.1, R45.2
- new net N$15: R45.1, U1.21
- new net QSPI_CSN: IC9.1, R46.2, R47.2, U1.56
- new net QSPI_SCLK: IC9.6, U1.52
- new net QSPI_SD0: IC9.5, U1.53
- new net QSPI_SD1: IC9.2, U1.55
- new net QSPI_SD2: IC9.3, U1.54
- new net QSPI_SD3: IC9.7, U1.51
- new net USB_VDD: U1.48
- new net VCC: C16.2, IC9.8, R46.1
- net GND: now also C14.1, C15.1, C16.1, IC9.4, U1.57
- net OFF_SW: now also R47.1

Commit message: ASAS
Parts:
- removed U1: RP2040, RP2040:QFN40P700X700X90-57N
- added C17, C18, C19, C20, C21, C22, C23, C26, C27: (no value), rcl:C0805
- added C24, C25: 1u, rcl:C0805
- added U$1: RP2040, jason_eagle6:QFN40P700X700X90-57N
Connections:
- removed net ADC_AVDD: U1.43
- removed net DVDD: U1.23, U1.50
- removed net IOVDD: U1.1, U1.10, U1.22, U1.33, U1.42, U1.49
- removed net USB_VDD: U1.48
- new net +1V1: C25.2, C26.2, C27.2, U$1.23, U$1.45, U$1.50
- new net +3V3: C17.2, C18.2, C19.2, C20.2, C21.2, C22.2, C23.2, C24.2, U$1.1, U$1.10, U$1.22, U$1.33, U$1.42, U$1.43, U$1.44, U$1.48, U$1.49
- new net N$44: U$1.19
- new net N$45: U$1.24
- new net N$46: U$1.25
- new net N$47: U$1.26
- new net N$65: U$1.37
- new net USB_DM: U$1.46
- new net USB_DP: U$1.47
- net AUXIN: now also U$1.30
- net AUXOUT: now also U$1.29
- net D_ADT: now also U$1.18
- net D_ARK: now also U$1.16
- net D_ENA: now also U$1.34
- net D_KCK: now also U$1.15, U$1.17
- net D_KDT: now also U$1.14
- net ENC1: now also U$1.2
- net ENC2: now also U$1.3
- net GATE1: now also U$1.9
- net GATE2: now also U$1.11
- net GATE3: now also U$1.12
- net GATE4: now also U$1.13
- net GND: now also C17.1, C18.1, C19.1, C20.1, C21.1, C22.1, C23.1, C24.1, C25.1, C26.1, C27.1, U$1.57; no longer U1.57
- net I2C0SCL: now also U$1.32
- net I2C0SDA: now also U$1.31
- net I2C1SCL: now also U$1.39
- net I2C1SDA: now also U$1.38
- net KEY_READ1: now also U$1.40
- net KEY_READ2: now also U$1.41
- net LED1: now also U$1.6
- net LED2: now also U$1.7
- net LED3: now also U$1.8
- net MIDIRX: now also U$1.28
- net MIDITX: now also U$1.27
- net N$10: now also U$1.20; no longer U1.20
- net N$15: now also U$1.21; no longer U1.21
- net OFF_SW: now also U$1.4
- net PWR_CTRL: now also U$1.5
- net QSPI_CSN: now also U$1.56; no longer U1.56
- net QSPI_SCLK: now also U$1.52; no longer U1.52
- net QSPI_SD0: now also U$1.53; no longer U1.53
- net QSPI_SD1: now also U$1.55; no longer U1.55
- net QSPI_SD2: now also U$1.54; no longer U1.54
- net QSPI_SD3: now also U$1.51; no longer U1.51
- net SYNCIN: now also U$1.35
- net SYNCOUT: now also U$1.36

Commit message: 3v3/rp2010
Parts:
- removed C1, C19, C21, C4: (no value), rcl:C0805
- removed C11, C2: 18p, rcl:C0805
- removed GD3: (no value), pinhead:1X01
- removed IC1: MKE02_44PIN, jason_eagle6:TQFP44
- removed PD6, PD7, PH2: TPTP17R, testpad:TP17R
- removed R5, R6: (no value), rcl:R0805
- removed XTL1: 20m, crystal:HC49/S
- added D+: (no value), pinhead:1X01
- added TP1, TP2: TPTP07SQ, testpad:TP07SQ
- C14, C15, C17, C18, C20, C22, C23, C24, C25, C26, C27: device rcl:C0805 -> rcl:C0603K
- C16: value 18p -> 100n; device rcl:C0805 -> resistor:C0603
- R45: device rcl:R0805 -> rcl:R0603
- moved C26 262.5 mm to (153.7, 76.5), flipped to the bottom, turned to 270 degrees
- moved C25 259.7 mm to (155.3, 76.5), flipped to the bottom, turned to 270 degrees
- moved C24 252.6 mm to (149.4, 78.9), flipped to the bottom
- moved C23 248.3 mm to (149.4, 77.1), flipped to the bottom
- moved C27 246.0 mm to (135.9, 66.8), flipped to the bottom, turned to 90 degrees
- moved C22 232.5 mm to (136.3, 73.2), flipped to the bottom, turned to 180 degrees
- moved C20 231.3 mm to (137.7, 79.6), flipped to the bottom, turned to 225 degrees
- moved R47 221.0 mm to (144.0, 87.6), flipped to the bottom, turned to 270 degrees
- moved C18 220.1 mm to (140.8, 65.2), flipped to the bottom, turned to 90 degrees
- moved C17 215.7 mm to (137.8, 66.8), flipped to the bottom, turned to 90 degrees
- moved U$1 215.5 mm to (143.5, 72.4), flipped to the bottom, turned to 225 degrees
- moved R46 214.5 mm to (142.2, 83.8), flipped to the bottom, turned to 180 degrees
- moved C15 208.4 mm to (154.3, 81.8), flipped to the bottom, turned to 315 degrees
- moved C14 202.8 mm to (147.7, 88.3), flipped to the bottom, turned to 135 degrees
- moved R45 198.1 mm to (149.4, 80.8), flipped to the bottom, turned to 180 degrees
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- renumbered GD5 to D-
Connections:
- removed net +5V: C1.2, C10.2, C12.+, C13.+, C3.2, C4.2, C5.2, C6.2, C7.2, C8.2, C9.2, IC1.28, IC1.5, IC1.6, IC2.8, IC3.10, IC3.16, IC4.10, IC4.16, IC5.10, IC5.16, IC6.10, IC6.16, IC7.1, IC7.7, IC8.1, IC8.7, R1.2, R2.2, R3.2, R4.2, R42.2, R43.2, R44.2, R5.2, VCC.1, VCC1.1, VCC2.1
- removed net N$44: U$1.19
- removed net N$45: U$1.24
- removed net N$46: U$1.25
- removed net N$47: U$1.26
- removed net NRESET: IC1.43, R3.1, RESET.1
- removed net PTD6: IC1.17, PD6.TP
- removed net PTD7: IC1.16, PD7.TP
- removed net PTH2: IC1.4, PH2.TP
- removed net SWDCLK: IC1.42, R5.1, SWD_CLK.1
- removed net SWDIO: IC1.44, R4.1, SWD_DAT.1
- removed net VCC: C16.2, IC9.8, R46.1
- new net N$25: D-.1, R4.2
- new net N$26: TP2.TP, U$1.19
- new net SWD_CLK: SWD_CLK.1, U$1.24
- new net SWD_DAT: SWD_DAT.1, U$1.25
- new net SWD_RESET: RESET.1, U$1.26
- net +3V3: now also C10.2, C12.+, C13.+, C16.2, C3.2, C5.2, C6.2, C7.2, C8.2, C9.2, IC2.8, IC3.10, IC3.16, IC4.10, IC4.16, IC5.10, IC5.16, IC6.10, IC6.16, IC7.1, IC7.7, IC8.1, IC8.7, IC9.8, R1.2, R2.2, R42.2, R43.2, R44.2, R46.1, VCC.1, VCC1.1; no longer C19.2, C21.2
- net AUXIN: now also U$1.41; no longer IC1.36, U$1.30
- net AUXOUT: now also U$1.3; no longer IC1.25, U$1.29
- net D_ACK: now also U$1.4; no longer IC1.22
- net D_ADT: now also U$1.7; no longer IC1.21, U$1.18
- net D_ARK: now also U$1.5; no longer IC1.20, U$1.16
- net D_ENA: now also U$1.6; no longer IC1.34, U$1.34
- net D_KCK: now also U$1.36; no longer IC1.19, U$1.15, U$1.17
- net D_KDT: now also U$1.35; no longer IC1.18, U$1.14
- net ENC1: now also U$1.31; no longer IC1.1, U$1.2
- net ENC2: now also U$1.30; no longer IC1.2, U$1.3
- net GATE1: now also U$1.14; no longer IC1.31, U$1.9
- net GATE2: now also U$1.13; no longer IC1.30, U$1.11
- net GATE3: no longer IC1.29
- net GATE4: now also U$1.11; no longer IC1.26, U$1.13
- net GND: no longer C1.1, C11.1, C19.1, C2.1, C21.1, C4.1, D-.1, GD3.1, IC1.11, IC1.27, IC1.8
- net I2C0SCL: now also U$1.16; no longer IC1.32, U$1.32
- net I2C0SDA: now also U$1.15; no longer IC1.33, U$1.31
- net I2C1SCL: no longer IC1.39
- net I2C1SDA: no longer IC1.40
- net KEY_READ1: now also U$1.34; no longer IC1.37, U$1.40
- net KEY_READ2: now also U$1.32; no longer IC1.13, U$1.41
- net LED1: now also U$1.27; no longer IC1.12, U$1.6
- net LED2: now also U$1.28; no longer IC1.14, U$1.7
- net LED3: now also U$1.29; no longer IC1.15, U$1.8
- net MIDIRX: now also U$1.9; no longer IC1.24, U$1.28
- net MIDITX: now also U$1.8; no longer IC1.23, U$1.27
- net N$4: now also VCC2.1; no longer C2.2, IC1.9, R6.2, XTL1.2
- net N$5: now also D+.1, R3.2; no longer C11.2, IC1.10, R6.1, XTL1.1
- net N$65: now also TP1.TP
- net OFF_SW: now also U$1.17; no longer IC1.3, U$1.4
- net PWR_CTRL: now also U$1.40; no longer IC1.38, U$1.5
- net SYNCIN: now also U$1.2; no longer IC1.35, U$1.35
- net SYNCOUT: now also U$1.18; no longer IC1.41, U$1.36
- net USB_DM: now also R4.1
- net USB_DP: now also R3.1
Routing:
- net +3V3: track 0.00 -> 541.1 mm, vias 0 -> 23
- net +5V: track 517.8 -> 0.00 mm, vias 18 -> 0
- net USB_DP: track 0.00 -> 64.4 mm, vias 0 -> 2
- net USB_DM: track 0.00 -> 59.1 mm, vias 0 -> 2
- net QSPI_CSN: track 0.00 -> 38.5 mm, vias 0 -> 4
- net AUXIN: track 10.8 -> 47.2 mm, vias 0 -> 1
- net PWR_CTRL: track 15.4 -> 47.2 mm, vias 0 -> 1
- net +1V1: track 0.00 -> 27.6 mm
- net KEY_READ1: track 246.7 -> 220.1 mm
- net SYNCIN: track 14.0 -> 33.9 mm, vias 0 -> 1
- net N$10: track 0.00 -> 19.2 mm
- net SWDIO: track 17.5 -> 0.00 mm, vias 1 -> 0
- net SWD_DAT: track 0.00 -> 17.4 mm
- net QSPI_SD1: track 0.00 -> 16.9 mm, vias 0 -> 2
- net AUXOUT: track 13.2 -> 28.9 mm, vias 0 -> 1
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
Commit message: Rolling back RP2040 changes
Parts:
- removed C14, C15: 18p, rcl:C0603K
- removed C16: 100n, resistor:C0603
- removed C17, C18, C20, C22, C23, C26, C27: (no value), rcl:C0603K
- removed C24, C25: 1u, rcl:C0603K
- removed D+: (no value), pinhead:1X01
- removed IC9: W25Q128, jason_eagle6:SO08
- removed Q1: (no value), adafruit:CTS406
- removed R45: (no value), rcl:R0603
- removed R46, R47: (no value), rcl:R0805
- removed TP1, TP2: TPTP07SQ, testpad:TP07SQ
- removed U$1: RP2040, jason_eagle6:QFN40P700X700X90-57N
- added C1, C4: (no value), rcl:C0805
- added C11, C2: 18p, rcl:C0805
- added GD3: (no value), pinhead:1X01
- added IC1: MKE02_44PIN, jason_eagle6:TQFP44
- added PD6, PD7, PH2: TPTP17R, testpad:TP17R
- added R5, R6: (no value), rcl:R0805
- added XTL1: 20m, crystal:HC49/S
- moved R3 34.7 mm to (150.0, 89.3), turned to 90 degrees
- moved R4 32.2 mm to (147.7, 89.3), turned to 90 degrees
- moved SWD_CLK 16.5 mm to (154.9, 86.4)
- moved SWD_DAT 16.5 mm to (154.9, 81.3)
- moved VCC2 16.5 mm to (154.9, 88.9)
- moved GD4 16.5 mm to (154.9, 78.7)
- moved RESET 16.5 mm to (154.9, 83.8)
- moved C3 13.1 mm to (136.5, 86.7), turned to 270 degrees
- moved R43 12.4 mm to (148.6, 94.7), turned to 180 degrees
- moved R44 8.81 mm to (148.6, 92.5), turned to 180 degrees
- moved R26 6.49 mm to (128.3, 64.8)
- moved GD1 3.59 mm to (123.2, 94.5)
- moved R1 2.34 mm to (128.7, 76.8)
- moved R2 2.09 mm to (128.7, 79.4)
- moved IC2 0.64 mm to (119.4, 77.5)
- renumbered D- to GD5
Connections:
- removed net +1V1: C25.2, C26.2, C27.2, U$1.23, U$1.45, U$1.50
- removed net +3V3: C10.2, C12.+, C13.+, C16.2, C17.2, C18.2, C20.2, C22.2, C23.2, C24.2, C3.2, C5.2, C6.2, C7.2, C8.2, C9.2, IC2.8, IC3.10, IC3.16, IC4.10, IC4.16, IC5.10, IC5.16, IC6.10, IC6.16, IC7.1, IC7.7, IC8.1, IC8.7, IC9.8, R1.2, R2.2, R42.2, R43.2, R44.2, R46.1, U$1.1, U$1.10, U$1.22, U$1.33, U$1.42, U$1.43, U$1.44, U$1.48, U$1.49, VCC.1, VCC1.1
- removed net N$10: C14.2, Q1.3, U$1.20
- removed net N$12: C15.2, Q1.1, R45.2
- removed net N$15: R45.1, U$1.21
- removed net N$25: GD5.1, R4.2
- removed net N$26: TP2.TP, U$1.19
- removed net N$65: TP1.TP, U$1.37
- removed net QSPI_CSN: IC9.1, R46.2, R47.2, U$1.56
- removed net QSPI_SCLK: IC9.6, U$1.52
- removed net QSPI_SD0: IC9.5, U$1.53
- removed net QSPI_SD1: IC9.2, U$1.55
- removed net QSPI_SD2: IC9.3, U$1.54
- removed net QSPI_SD3: IC9.7, U$1.51
- removed net SWD_CLK: SWD_CLK.1, U$1.24
- removed net SWD_DAT: SWD_DAT.1, U$1.25
- removed net SWD_RESET: RESET.1, U$1.26
- removed net USB_DM: R4.1, U$1.46
- removed net USB_DP: R3.1, U$1.47
- new net +5V: C1.2, C10.2, C12.+, C13.+, C3.2, C4.2, C5.2, C6.2, C7.2, C8.2, C9.2, IC1.28, IC1.5, IC1.6, IC2.8, IC3.10, IC3.16, IC4.10, IC4.16, IC5.10, IC5.16, IC6.10, IC6.16, IC7.1, IC7.7, IC8.1, IC8.7, R1.2, R2.2, R3.2, R4.2, R42.2, R43.2, R44.2, R5.2, VCC.1, VCC1.1, VCC2.1
- new net NRESET: IC1.43, R3.1, RESET.1
- new net PTD6: IC1.17, PD6.TP
- new net PTD7: IC1.16, PD7.TP
- new net PTH2: IC1.4, PH2.TP
- new net SWDCLK: IC1.42, R5.1, SWD_CLK.1
- new net SWDIO: IC1.44, R4.1, SWD_DAT.1
- net AUXIN: now also IC1.36; no longer U$1.41
- net AUXOUT: now also IC1.25; no longer U$1.3
- net D_ACK: now also IC1.22; no longer U$1.4
- net D_ADT: now also IC1.21; no longer U$1.7
- net D_ARK: now also IC1.20; no longer U$1.5
- net D_ENA: now also IC1.34; no longer U$1.6
- net D_KCK: now also IC1.19; no longer U$1.36
- net D_KDT: now also IC1.18; no longer U$1.35
- net ENC1: now also IC1.1; no longer U$1.31
- net ENC2: now also IC1.2; no longer U$1.30
- net GATE1: now also IC1.31; no longer U$1.14
- net GATE2: now also IC1.30; no longer U$1.13
- net GATE3: now also IC1.29; no longer U$1.12
- net GATE4: now also IC1.26; no longer U$1.11
- net GND: now also C1.1, C11.1, C2.1, C4.1, GD3.1, GD5.1, IC1.11, IC1.27, IC1.8; no longer C14.1, C15.1, C16.1, C17.1, C18.1, C20.1, C22.1, C23.1, C24.1, C25.1, C26.1, C27.1, IC9.4, U$1.57
- net I2C0SCL: now also IC1.32; no longer U$1.16
- net I2C0SDA: now also IC1.33; no longer U$1.15
- net I2C1SCL: now also IC1.39; no longer U$1.39
- net I2C1SDA: now also IC1.40; no longer U$1.38
- net KEY_READ1: now also IC1.37; no longer U$1.34
- net KEY_READ2: now also IC1.13; no longer U$1.32
- net LED1: now also IC1.12; no longer U$1.27
- net LED2: now also IC1.14; no longer U$1.28
- net LED3: now also IC1.15; no longer U$1.29
- net MIDIRX: now also IC1.24; no longer U$1.9
- net MIDITX: now also IC1.23; no longer U$1.8
- net N$4: now also C2.2, IC1.9, R6.2, XTL1.2; no longer VCC2.1
- net N$5: now also C11.2, IC1.10, R6.1, XTL1.1; no longer D+.1, R3.2
- net OFF_SW: now also IC1.3; no longer R47.1, U$1.17
- net PWR_CTRL: now also IC1.38; no longer U$1.40
- net SYNCIN: now also IC1.35; no longer U$1.2
- net SYNCOUT: now also IC1.41; no longer U$1.18
Routing:
- net +3V3: track 541.1 -> 0.00 mm, vias 23 -> 0
- net +5V: track 0.00 -> 517.8 mm, vias 0 -> 18
- net USB_DP: track 64.4 -> 0.00 mm, vias 2 -> 0
- net USB_DM: track 59.1 -> 0.00 mm, vias 2 -> 0
- net QSPI_CSN: track 38.5 -> 0.00 mm, vias 4 -> 0
- net AUXIN: track 47.2 -> 10.8 mm, vias 1 -> 0
- net PWR_CTRL: track 47.2 -> 15.4 mm, vias 1 -> 0
- net +1V1: track 27.6 -> 0.00 mm
- net KEY_READ1: track 220.1 -> 246.7 mm
- net SYNCIN: track 33.9 -> 14.0 mm, vias 1 -> 0
- net N$10: track 19.2 -> 0.00 mm
- net SWDIO: track 0.00 -> 17.5 mm, vias 0 -> 1
- net SWD_DAT: track 17.4 -> 0.00 mm
- net QSPI_SD1: track 16.9 -> 0.00 mm, vias 2 -> 0
- net AUXOUT: track 28.9 -> 13.2 mm, vias 1 -> 0
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