File: matrix_main_board.brd (EAGLE design)
At the start: 155.7 x 92.3 mm, 128 parts, among them IC1 MKE02_44PIN, IC2 24AA01SM, IC3 74HC595D, IC4 74HC595D, IC5 74HC595D, IC6 74HC595D, IC7 NPIC6C596, IC8 NPIC6C596

Commit message: in prog
Parts:
- added U$1: MKE02_64PIN64, jason_eagle6:TQFP64
Connections:
- removed net PTD6: IC1.17, PD6.TP
- removed net PTD7: IC1.16, PD7.TP
- new net N$10: PD7.TP, U$1.22
- new net N$12: PD6.TP, U$1.23
- net +5V: now also U$1.41, U$1.7, U$1.8
- net AUXIN: now also U$1.51
- net AUXOUT: now also U$1.37
- net D_ACK: now also U$1.32
- net D_ADT: now also U$1.31
- net D_ARK: now also U$1.26
- net D_ENA: now also U$1.49
- net D_KCK: now also U$1.25
- net D_KDT: now also U$1.24
- net ENC1: now also U$1.1
- net ENC2: now also U$1.2
- net GATE1: now also U$1.46
- net GATE2: now also U$1.45
- net GATE3: now also U$1.44
- net GATE4: now also U$1.38
- net GND: now also U$1.10, U$1.13, U$1.40
- net I2C0SCL: now also U$1.47
- net I2C0SDA: now also U$1.48
- net I2C1SCL: now also U$1.59
- net I2C1SDA: now also U$1.60
- net KEY_READ1: now also U$1.52
- net KEY_READ2: now also U$1.19
- net LED1: now also U$1.18
- net LED2: now also U$1.20
- net LED3: now also U$1.21
- net MIDIRX: now also U$1.34
- net MIDITX: now also U$1.33
- net N$4: now also U$1.11; no longer IC1.9
- net N$5: now also U$1.12; no longer IC1.10
- net NRESET: now also U$1.63; no longer IC1.43
- net OFF_SW: now also U$1.5
- net PTH2: now also U$1.6; no longer IC1.4
- net PWR_CTRL: now also U$1.54
- net SWDCLK: now also U$1.62; no longer IC1.42
- net SWDIO: now also U$1.64; no longer IC1.44
- net SYNCIN: now also U$1.50
- net SYNCOUT: now also U$1.61
Routing:
- net PTD7: track 8.45 -> 0.00 mm
- net PTH2: track 7.49 -> 0.00 mm
- net PTD6: track 6.25 -> 0.00 mm
- net +5V: track 517.8 -> 515.5 mm

Commit message: work in prog
Parts:
- removed IC1: MKE02_44PIN, jason_eagle6:TQFP44
- moved PD6 4.59 mm to (134.2, 65.3)
- moved XTL1 2.54 mm to (147.3, 66.0)
- moved C11 1.80 mm to (149.7, 62.5)
- moved R6 1.80 mm to (151.6, 65.0)
- moved C1 1.80 mm to (150.7, 71.9)
- moved C2 1.80 mm to (153.7, 67.4)
- moved C3 1.37 mm to (135.3, 87.5)
- moved PH2 1.27 mm to (154.9, 72.6)
- moved PD7 0.89 mm to (135.5, 67.3)
Connections:
- net +5V: no longer IC1.28, IC1.5, IC1.6
- net AUXIN: no longer IC1.36
- net AUXOUT: no longer IC1.25
- net D_ACK: no longer IC1.22
- net D_ADT: no longer IC1.21
- net D_ARK: no longer IC1.20
- net D_ENA: no longer IC1.34
- net D_KCK: no longer IC1.19
- net D_KDT: no longer IC1.18
- net ENC1: no longer IC1.1
- net ENC2: no longer IC1.2
- net GATE1: no longer IC1.31
- net GATE2: no longer IC1.30
- net GATE3: no longer IC1.29
- net GATE4: no longer IC1.26
- net GND: no longer IC1.11, IC1.27, IC1.8
- net I2C0SCL: no longer IC1.32
- net I2C0SDA: no longer IC1.33
- net I2C1SCL: no longer IC1.39
- net I2C1SDA: no longer IC1.40
- net KEY_READ1: no longer IC1.37
- net KEY_READ2: no longer IC1.13
- net LED1: no longer IC1.12
- net LED2: no longer IC1.14
- net LED3: no longer IC1.15
- net MIDIRX: no longer IC1.24
- net MIDITX: no longer IC1.23
- net OFF_SW: no longer IC1.3
- net PWR_CTRL: no longer IC1.38
- net SYNCIN: no longer IC1.35
- net SYNCOUT: no longer IC1.41
Routing:
- net D_ENA: track 163.7 -> 150.2 mm, vias 11 -> 10
- net N$5: track 13.3 -> 0.00 mm
- net N$4: track 11.0 -> 0.00 mm
- net N$12: track 0.00 -> 8.53 mm
- net N$10: track 0.00 -> 5.64 mm
- net +5V: track 515.5 -> 519.4 mm, vias 18 -> 19
- net KEY_READ2: track 47.2 -> 44.2 mm
- net LED3: track 16.5 -> 13.5 mm
- net LED1: track 24.8 -> 22.0 mm
- net LED2: track 21.4 -> 18.6 mm
- net GATE1: track 9.79 -> 6.99 mm
- net GATE3: track 12.0 -> 9.22 mm
- net GATE2: track 14.4 -> 11.6 mm
- net I2C0SCL: track 24.9 -> 22.1 mm
- net I2C0SDA: track 18.0 -> 15.3 mm
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
Commit message: 64pin
Parts:
- removed R3, R4, R5: (no value), rcl:R0805
- added PE6, PF4, PF5, PF6, PF7, PG0, PG1, PG2, PH0, PH1, PH6, PH7: TPTP17R, testpad:TP17R
- moved C11 0.65 mm to (150.4, 62.6)
- moved C2 0.57 mm to (154.2, 67.7)
- moved R6 0.28 mm to (151.4, 65.2)
- renumbered GD4 to GD, RESET to RT, SWD_CLK to CK, SWD_DAT to DT, U$1 to IC1, VCC2 to VC
Connections:
- new net N$15: IC1.27, PF7.TP
- new net N$25: IC1.28, PF6.TP
- new net N$26: IC1.29, PF5.TP
- new net N$27: IC1.30, PF4.TP
- new net N$36: IC1.14, PH1.TP
- new net N$37: IC1.15, PH0.TP
- new net N$38: IC1.16, PE6.TP
- new net N$41: IC1.4, PH6.TP
- new net N$43: IC1.57, PG1.TP
- new net PG0: IC1.58, PG0.TP
- new net PTG2: IC1.56, PG2.TP
- new net PTH7: IC1.3, PH7.TP
- net +5V: no longer R3.2, R4.2, R5.2
- net NRESET: no longer R3.1
- net SWDCLK: no longer R5.1
- net SWDIO: no longer R4.1
Routing:
- net D_ENA: track 150.2 -> 166.9 mm, vias 10 -> 9
- net N$5: track 0.00 -> 15.3 mm
- net SWDIO: track 17.4 -> 3.55 mm, vias 1 -> 0
- net N$4: track 0.00 -> 13.1 mm
- net NRESET: track 15.3 -> 5.31 mm, vias 1 -> 0
- net N$15: track 0.00 -> 9.17 mm, vias 0 -> 1
- net N$25: track 0.00 -> 7.00 mm, vias 0 -> 1
- net PTH2: track 0.00 -> 6.65 mm
- net N$37: track 0.00 -> 5.91 mm, vias 0 -> 1
- net SWDCLK: track 12.7 -> 6.91 mm
- net N$38: track 0.00 -> 5.22 mm, vias 0 -> 1
- net N$36: track 0.00 -> 4.56 mm, vias 0 -> 1
- net N$26: track 0.00 -> 4.39 mm, vias 0 -> 1
- net N$41: track 0.00 -> 4.37 mm, vias 0 -> 1
- net ENC1: track 75.5 -> 79.8 mm
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Other:
- board text added: "NOODLEBOX Main Board v4"
- board text removed: "NOODLEBOX Main Board v3"

Commit message: correct footprint
Parts:
- IC1: value MKE02_64PIN64 -> MKE02_64PINQFP64; device jason_eagle6:TQFP64 -> jason_eagle6:QFP64_SOT393
- moved C1 1.27 mm to (150.7, 70.6)
- moved PD6 1.27 mm to (134.2, 64.0)
- moved PD7 1.20 mm to (134.9, 66.3)
- moved PG2 1.02 mm to (149.0, 87.0)
- moved PH2 0.92 mm to (155.2, 71.8)
- moved PG0 0.77 mm to (150.2, 85.3)
- moved PH7 0.52 mm to (152.9, 75.2)
- moved C3 0.51 mm to (134.8, 87.5)
- turned IC1 to 315 degrees
Routing:
- net N$12: track 8.53 -> 10.2 mm
- net SYNCOUT: track 14.7 -> 15.9 mm
- net I2C0SCL: track 22.1 -> 21.0 mm
- net GATE2: track 11.6 -> 10.5 mm
- net GATE1: track 6.99 -> 5.93 mm
- net OFF_SW: track 31.1 -> 32.0 mm
- net PTH2: track 6.65 -> 7.62 mm
- net GATE3: track 9.22 -> 8.30 mm
- net N$10: track 5.64 -> 6.56 mm
- net LED2: track 18.6 -> 19.5 mm
- net PTH7: track 2.52 -> 3.39 mm
- net PTG2: track 2.23 -> 3.09 mm
- net LED3: track 13.5 -> 14.2 mm
- net KEY_READ2: track 44.2 -> 44.9 mm
- net PG0: track 2.06 -> 2.64 mm
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Other:
- board text added: "NOODLEBOX Main Board v5"
- board text removed: "NOODLEBOX Main Board v4"
